Commit message: changed urdf and added a new config
urdf with tcp link
new moveit config with the tcp

File: yumi_description/urdf/.ipynb_checkpoints/yumi-checkpoint.urdf (robot description, URDF)
Before this commit: robot yumi, 24 links, 23 joints
Links:
- removed link tcp_link_l
Joints:
- removed joint joint_tcp_l
- joint joint_tcp_r: origin xyz=0 0 0.135 rpy=0 0 0 -> xyz=0 0 0.1 rpy=0 0 0
